Commit message: Made some slight change

File: description/gazebo_controller.xacro (robot description, xacro)
@@ -1,4 +1,5 @@
 <?xml version="1.0"?>
 <robot xmlns:xacro="http://www.ros.org/wiki/xacro">
+   <!-- Two Differential-drive plugin  -->
     <gazebo>
         <plugin name="diff_drive_robot_plugin" filename="libgazebo_ros_diff_drive.so">

File: description/robot.urdf.xacro (robot description, xacro)
@@ -5,3 +5,5 @@
   <!-- The gazebo control file  -->
   <xacro:include filename="gazebo_controller.xacro"/>
+  <!-- The lidar sensor file  -->
+  <xacro:include filename="lidar_sensor.xacro"/>
 </robot>

File: description/robot.xacro (robot description, xacro)
@@ -129,36 +129,3 @@
       <mu2 value="0.100"/>
     </gazebo>
-  <!-- LIDAR SENSOR JOINT  -->
-    <joint name="laser_joint" type="fixed">
-        <parent link="chassis"/>
-        <child link="laser_frame"/>
-        <origin xyz="0.122 0 0.212" rpy="0 0 0"/>
-    </joint>
-    <link name="laser_frame">
-        <visual>
-            <geometry>
-                <cylinder radius="0.05" length="0.04"/>
-            </geometry>
-            <material name="black"/>
-        </visual>
-        <visual>
-            <origin xyz="0 0 -0.05"/>
-            <geometry>
-                <cylinder radius="0.01" length="0.1"/>
-            </geometry>
-            <material name="black"/>
-        </visual>
-        <collision>
-            <geometry>
-                <cylinder radius="0.05" length="0.04"/>
-            </geometry>
-        </collision>
-        <xacro:inertial_cylinder mass="0.1" length="0.04" radius="0.05">
-            <origin xyz="0 0 0" rpy="0 0 0"/>
-        </xacro:inertial_cylinder>
-    </link>
-    <!-- We put colour to our lidar here  -->
-    <gazebo reference="laser_frame">
-    <material>Gazebo/Blue</material>
-    </gazebo>
 </robot>
