Commit message: Added an inertial file

File: description/robot.xacro (robot description, xacro)
@@ -1,4 +1,5 @@
 <?xml version="1.0"?>
 <robot xmlns:xacro="http://www.ros.org/wiki/xacro" name="robot">
+<xacro:include filename="inertial.xacro"/>
  <!-- Setting the meshes colour  -->
 <!-- white -->
@@ -21,4 +22,5 @@
 <link name="base_link">
 </link>
+<!-- link to the chassis  -->
 <joint name="chassis_joint" type="fixed">
     <parent link="base_link"/>
@@ -35,4 +37,85 @@
         <material name="orange"/>
     </visual>
+    <collusion>
+        <origin xyz="0.15 0 0.075"/>
+        <geometry>
+            <box size="0.3 0.3 0.15"/>
+        </geometry>
+    </collusion>
+    <xacro:inertial_box mass="0.5" x="0.3" y="0.3" z="0.15">
+     <origin xyz="0.15 0 0.075" rpy="0 0 0"/>
+    </xacro:inertial_box>
+</link>
+<!-- The left wheel link  -->
+<joint name="left_wheel_joint" type="continuous">
+  <parent link="base_link"/>
+  <child link="left_wheel"/>
+  <origin xyz="0 0.175 0" rpy="-${pi/2} 0 0"/>
+  <axis xyz="0 0 1"/>
+</joint>
+<link name="left_wheel">
+ <visual>
+    <geometry>
+       <cylinder radius="0.05" length="0.04"/>
+    </geometry>
+    <material name="black"/>
+ </visual>
+ <collusion>
+    <geometry>
+       <cylinder radius="0.05" length="0.04"/>
+    </geometry>
+    <material name="black"/>
+ </collusion>
+ <xacro:inertial_cylinder mass="0.1" length="0.04" radius="0.05">
+  <origin xyz="0 0 0" rpy="0 0 0"/>
+ </xacro:inertial_cylinder>
+</link>
+<!-- The right wheel link  -->
+<joint name="right_wheel_joint" type="continuous">
+  <parent link="base_link"/>
+  <child link="right_wheel"/>
+  <origin xyz="0 -0.175 0" rpy="${pi/2} 0 0"/>
+  <axis xyz="0 0 -1"/>
+</joint>
+<link name="right_wheel">
+ <visual>
+    <geometry>
+       <cylinder radius="0.05" length="0.04"/>
+    </geometry>
+    <material name="black"/>
+ </visual>
+ <collusion>
+    <geometry>
+       <cylinder radius="0.05" length="0.04"/>
+    </geometry>
+ </collusion>
+ <xacro:inertial_cylinder mass="0.1" length="0.04" radius="0.05">
+  <origin xyz="0 0 0" rpy="0 0 0"/>
+ </xacro:inertial_cylinder>
+</link>
+<!-- dolly wheel link  -->
+<joint name="dolly_wheel_joint" type="fixed">
+ <parent link="chassis"/>
+ <child link="dolly_wheel"/>
+ <origin xyz="0.24 0 0"/>
+</joint>
+<link name="dolly_wheel">
+<visual>
+ <geometry>
+   <sphere radius="0.05"/>
+ </geometry>
+ <!-- give it a colour -->
+ <material name="black"/>
+</visual>
+<collusion>
+ <geometry>
+   <sphere radius="0.05"/>
+ </geometry>
+ <!-- give it a colour -->
+ <material name="black"/>
+</collusion>
+<xacro:inertial_sphere mass="0.1"  radius="0.05">
+  <origin xyz="0 0 0" rpy="0 0 0"/>
+ </xacro:inertial_sphere>
 </link>
 </robot>

Commit message: Added some xacro xml tags

File: description/robot.xacro (robot description, xacro)
@@ -1,121 +1,111 @@
 <?xml version="1.0"?>
-<robot xmlns:xacro="http://www.ros.org/wiki/xacro" name="robot">
-<xacro:include filename="inertial.xacro"/>
- <!-- Setting the meshes colour  -->
-<!-- white -->
- <material name="white">
-    <color rgba="1 1 1 1" />
- </material>
- <!-- orange -->
- <material name="orange">
-    <color rgba="1 0.3 0.1 1" />
- </material>
- <!-- blue -->
- <material name="blue">
-    <color rgba="0.2 0.2 1 1" />
- </material>
- <!-- black -->
- <material name="black">
-    <color rgba="0 0 0 1" />
- </material>
-<!-- The link to the centre of the robot (called it "base_link") -->
-<link name="base_link">
-</link>
-<!-- link to the chassis  -->
-<joint name="chassis_joint" type="fixed">
-    <parent link="base_link"/>
-    <child link="chassis"/>
-<!-- We want the origin of the chassis sitting at the back/centre of the chassis -->
-    <origin xyz="-0.1 0 0"/>
-</joint>
-<link name="chassis">
-    <visual>
-        <origin xyz="0.15 0 0.075"/>
-        <geometry>
-            <box size="0.3 0.3 0.15"/>
-        </geometry>
-        <material name="orange"/>
-    </visual>
-    <collusion>
-        <origin xyz="0.15 0 0.075"/>
-        <geometry>
-            <box size="0.3 0.3 0.15"/>
-        </geometry>
-    </collusion>
-    <xacro:inertial_box mass="0.5" x="0.3" y="0.3" z="0.15">
-     <origin xyz="0.15 0 0.075" rpy="0 0 0"/>
-    </xacro:inertial_box>
-</link>
-<!-- The left wheel link  -->
-<joint name="left_wheel_joint" type="continuous">
-  <parent link="base_link"/>
-  <child link="left_wheel"/>
-  <origin xyz="0 0.175 0" rpy="-${pi/2} 0 0"/>
-  <axis xyz="0 0 1"/>
-</joint>
-<link name="left_wheel">
- <visual>
-    <geometry>
-       <cylinder radius="0.05" length="0.04"/>
-    </geometry>
-    <material name="black"/>
- </visual>
- <collusion>
-    <geometry>
-       <cylinder radius="0.05" length="0.04"/>
-    </geometry>
-    <material name="black"/>
- </collusion>
- <xacro:inertial_cylinder mass="0.1" length="0.04" radius="0.05">
-  <origin xyz="0 0 0" rpy="0 0 0"/>
- </xacro:inertial_cylinder>
-</link>
-<!-- The right wheel link  -->
-<joint name="right_wheel_joint" type="continuous">
-  <parent link="base_link"/>
-  <child link="right_wheel"/>
-  <origin xyz="0 -0.175 0" rpy="${pi/2} 0 0"/>
-  <axis xyz="0 0 -1"/>
-</joint>
-<link name="right_wheel">
- <visual>
-    <geometry>
-       <cylinder radius="0.05" length="0.04"/>
-    </geometry>
-    <material name="black"/>
- </visual>
- <collusion>
-    <geometry>
-       <cylinder radius="0.05" length="0.04"/>
-    </geometry>
- </collusion>
- <xacro:inertial_cylinder mass="0.1" length="0.04" radius="0.05">
-  <origin xyz="0 0 0" rpy="0 0 0"/>
- </xacro:inertial_cylinder>
-</link>
-<!-- dolly wheel link  -->
-<joint name="dolly_wheel_joint" type="fixed">
- <parent link="chassis"/>
- <child link="dolly_wheel"/>
- <origin xyz="0.24 0 0"/>
-</joint>
-<link name="dolly_wheel">
-<visual>
- <geometry>
-   <sphere radius="0.05"/>
- </geometry>
- <!-- give it a colour -->
- <material name="black"/>
-</visual>
-<collusion>
- <geometry>
-   <sphere radius="0.05"/>
- </geometry>
- <!-- give it a colour -->
- <material name="black"/>
-</collusion>
-<xacro:inertial_sphere mass="0.1"  radius="0.05">
-  <origin xyz="0 0 0" rpy="0 0 0"/>
- </xacro:inertial_sphere>
-</link>
+<robot xmlns:xacro="http://www.ros.org/wiki/xacro" >
+    <xacro:include filename="inertial.xacro"/>
+    <material name="white">
+        <color rgba="1 1 1 1" />
+    </material>
+    <material name="orange">
+        <color rgba="1 0.3 0.1 1"/>
+    </material>
+    <material name="blue">
+        <color rgba="0.2 0.2 1 1"/>
+    </material>
+    <material name="black">
+        <color rgba="0 0 0 1"/>
+    </material>
+    <!-- BASE LINK -->
+    <link name="base_link">
+    </link>
+    <!-- CHASSIS LINK -->
+    <joint name="chassis_joint" type="fixed">
+        <parent link="base_link"/>
+        <child link="chassis"/>
+        <origin xyz="-0.1 0 0"/>
+    </joint>
+    <link name="chassis">
+        <visual>
+            <origin xyz="0.15 0 0.075"/>
+            <geometry>
+                <box size="0.3 0.3 0.15"/>
+            </geometry>
+            <material name="orange"/>
+        </visual>
+        <collision>
+            <origin xyz="0.15 0 0.075"/>
+            <geometry>
+                <box size="0.3 0.3 0.15"/>
+            </geometry>
+        </collision>
+        <xacro:inertial_box mass="0.5" x="0.3" y="0.3" z="0.15">
+            <origin xyz="0.15 0 0.075" rpy="0 0 0"/>
+        </xacro:inertial_box>
+    </link>
+    <!-- LEFT WHEEL OF ROBOT -->
+    <joint name="left_wheel_joint" type="continuous">
+        <parent link="base_link"/>
+        <child link="left_wheel"/>
+        <origin xyz="0 0.175 0" rpy="-${pi/2} 0 0" />
+        <axis xyz="0 0 1"/>
+    </joint>
+    <link name="left_wheel">
+        <visual>
+            <geometry>
+                <cylinder radius="0.05" length="0.04"/>
+            </geometry>
+            <material name="black"/>
+        </visual>
+        <collision>
+            <geometry>
+                <cylinder radius="0.05" length="0.04"/>
+            </geometry>
+        </collision>
+        <xacro:inertial_cylinder mass="0.1" length="0.04" radius="0.05">
+            <origin xyz="0 0 0" rpy="0 0 0"/>
+        </xacro:inertial_cylinder>
+    </link>
+    <!-- RIGHT WHEEL OF ROBOT -->
+    <joint name="right_wheel_joint" type="continuous">
+        <parent link="base_link"/>
+        <child link="right_wheel"/>
+        <origin xyz="0 -0.175 0" rpy="${pi/2} 0 0" />
+        <axis xyz="0 0 -1"/>
+    </joint>
+    <link name="right_wheel">
+        <visual>
+            <geometry>
+                <cylinder radius="0.05" length="0.04"/>
+            </geometry>
+            <material name="black"/>
+        </visual>
+        <collision>
+            <geometry>
+                <cylinder radius="0.05" length="0.04"/>
+            </geometry>
+        </collision>
+        <xacro:inertial_cylinder mass="0.1" length="0.04" radius="0.05">
+            <origin xyz="0 0 0" rpy="0 0 0"/>
+        </xacro:inertial_cylinder>
+    </link>
+    <!-- DOLLY WHEEEL JOINT -->
+    <joint name="dolly_wheel_joint" type="fixed">
+        <parent link="chassis"/>
+        <child link="dolly_wheel"/>
+        <origin xyz="0.24 0 0"/>
+    </joint>
+    <link name="dolly_wheel">
+        <visual>
+            <geometry>
+                <sphere radius="0.05"/>
+            </geometry>
+            <material name="black"/>
+        </visual>
+        <collision>
+            <geometry>
+                <sphere radius="0.05"/>
+            </geometry>
+        </collision>
+        <xacro:inertial_sphere mass="0.1" radius="0.05">
+            <origin xyz="0 0 0" rpy="0 0 0"/>
+        </xacro:inertial_sphere>
+    </link>
 </robot>

Commit message: Added mu1 and mu2 tags for friction of the dolly wheels

File: description/robot.xacro (robot description, xacro)
@@ -47,6 +47,6 @@
    <!-- Adding colour/fixing the colours to our urdf robot -->
     <!-- chassis link colour (Adding chassis link colour) -->
-    <gazebo reference="chassis_joint">
-      <material>Gazebo/orange</material>
+    <gazebo reference="chassis">
+      <material>Gazebo/Orange</material>
     </gazebo>
     <!-- LEFT WHEEL OF ROBOT -->
@@ -74,5 +74,5 @@
     </link>
     <gazebo reference="left_wheel">
-      <material>Gazebo/black</material>
+      <material>Gazebo/Black</material>
     </gazebo>
     <!-- RIGHT WHEEL OF ROBOT -->
@@ -100,5 +100,5 @@
     </link>
      <gazebo reference="right_wheel">
-      <material>Gazebo/black</material>
+      <material>Gazebo/Black</material>
     </gazebo>
     <!-- DOLLY WHEEEL JOINT -->
@@ -125,5 +125,7 @@
     </link>
      <gazebo reference="dolly_wheel">
-      <material>Gazebo/black</material>
+      <material>Gazebo/Black</material>
+      <mu1 value="0.100"/>
+      <mu2 value="0.100"/>
     </gazebo>
 </robot>

Commit message: Added a Lidar sensor

File: description/robot.xacro (robot description, xacro)
@@ -129,3 +129,36 @@
       <mu2 value="0.100"/>
     </gazebo>
+  <!-- LIDAR SENSOR JOINT  -->
+    <joint name="laser_joint" type="fixed">
+        <parent link="chassis"/>
+        <child link="laser_frame"/>
+        <origin xyz="0.122 0 0.212" rpy="0 0 0"/>
+    </joint>
+    <link name="laser_frame">
+        <visual>
+            <geometry>
+                <cylinder radius="0.05" length="0.04"/>
+            </geometry>
+            <material name="black"/>
+        </visual>
+        <visual>
+            <origin xyz="0 0 -0.05"/>
+            <geometry>
+                <cylinder radius="0.01" length="0.1"/>
+            </geometry>
+            <material name="black"/>
+        </visual>
+        <collision>
+            <geometry>
+                <cylinder radius="0.05" length="0.04"/>
+            </geometry>
+        </collision>
+        <xacro:inertial_cylinder mass="0.1" length="0.04" radius="0.05">
+            <origin xyz="0 0 0" rpy="0 0 0"/>
+        </xacro:inertial_cylinder>
+    </link>
+    <!-- We put colour to our lidar here  -->
+    <gazebo reference="laser_frame">
+    <material>Gazebo/Blue</material>
+    </gazebo>
 </robot>

Commit message: Made changes in the robot.xacro file

File: description/robot.xacro (robot description, xacro)
@@ -2,8 +2,4 @@
 <robot xmlns:xacro="http://www.ros.org/wiki/xacro" >
     <xacro:include filename="inertial.xacro"/>
-    <!-- <xacro:property name="chasis_color" value="Gazebo/orange"/>
-    <xacro:property name="tyre_color" value="Gazebo/black"/>
-    <xacro:property name="dolly_color" value="Gazebo/black"/>
-    <xacro:property name="wheel_color" value="Gazebo/black"/> -->
     <material name="white">
         <color rgba="1 1 1 1" />
