Commit message: Changes made

File: description/lidar_sensor.xacro (robot description, xacro)
@@ -30,5 +30,5 @@
         </xacro:inertial_cylinder>
     </link>
-    We put colour to our lidar here
+    <!-- We put colour to our lidar here  -->
     <gazebo reference="laser_frame">
     <material>Gazebo/Blue</material>

File: description/robot.xacro (robot description, xacro)
@@ -29,5 +29,5 @@
                 <box size="0.3 0.3 0.15"/>
             </geometry>
-            <material name="orange"/>
+            <material name="blue"/>
         </visual>
         <collision>
@@ -44,5 +44,5 @@
     <!-- chassis link colour (Adding chassis link colour) -->
     <gazebo reference="chassis">
-      <material>Gazebo/Orange</material>
+      <material>Gazebo/Blue</material>
     </gazebo>
     <!-- LEFT WHEEL OF ROBOT -->
