Commit message: Added a robot.xacro file

File: description/robot.urdf.xacro (robot description, xacro)
@@ -1,5 +1,4 @@
 <?xml version="1.0"?>
 <robot xmlns:xacro="http://www.ros.org/wiki/xacro" name="robot">
-<!-- Example link -->
-<link name="base_link"></link>
+  <xacro:include filename="robot.xacro"/>
 </robot>

Commit message: Gazebo plugin file

File: description/robot.urdf.xacro (robot description, xacro)
@@ -1,4 +1,7 @@
 <?xml version="1.0"?>
 <robot xmlns:xacro="http://www.ros.org/wiki/xacro" name="robot">
+  <!-- The robot .xacro file  -->
   <xacro:include filename="robot.xacro"/>
+  <!-- The gazebo control file  -->
+  <xacro:include filename="gazebo_controller.xacro"/>
 </robot>

File: description/robot.xacro (robot description, xacro)
@@ -2,4 +2,8 @@
 <robot xmlns:xacro="http://www.ros.org/wiki/xacro" >
     <xacro:include filename="inertial.xacro"/>
+    <!-- <xacro:property name="chasis_color" value="Gazebo/orange"/>
+    <xacro:property name="tyre_color" value="Gazebo/black"/>
+    <xacro:property name="dolly_color" value="Gazebo/black"/>
+    <xacro:property name="wheel_color" value="Gazebo/black"/> -->
     <material name="white">
         <color rgba="1 1 1 1" />
@@ -41,4 +45,9 @@
         </xacro:inertial_box>
     </link>
+   <!-- Adding colour/fixing the colours to our urdf robot -->
+    <!-- chassis link colour (Adding chassis link colour) -->
+    <gazebo reference="chassis_joint">
+      <material>Gazebo/orange</material>
+    </gazebo>
     <!-- LEFT WHEEL OF ROBOT -->
     <joint name="left_wheel_joint" type="continuous">
@@ -64,4 +73,7 @@
         </xacro:inertial_cylinder>
     </link>
+    <gazebo reference="left_wheel">
+      <material>Gazebo/black</material>
+    </gazebo>
     <!-- RIGHT WHEEL OF ROBOT -->
     <joint name="right_wheel_joint" type="continuous">
@@ -87,4 +99,7 @@
         </xacro:inertial_cylinder>
     </link>
+     <gazebo reference="right_wheel">
+      <material>Gazebo/black</material>
+    </gazebo>
     <!-- DOLLY WHEEEL JOINT -->
     <joint name="dolly_wheel_joint" type="fixed">
@@ -97,5 +112,5 @@
             <geometry>
                 <sphere radius="0.05"/>
-            </geometry>
+            </geometry>`
             <material name="black"/>
         </visual>
@@ -109,3 +124,6 @@
         </xacro:inertial_sphere>
     </link>
+     <gazebo reference="dolly_wheel">
+      <material>Gazebo/black</material>
+    </gazebo>
 </robot>

Commit message: Added files

File: description/robot.urdf.xacro (robot description, xacro)
@@ -6,5 +6,5 @@
   <xacro:include filename="gazebo_controller.xacro"/>
   <!-- The lidar sensor file  -->
-  <!-- <xacro:include filename="lidar_sensor.xacro"/> -->
+  <xacro:include filename="lidar_sensor.xacro"/>
   <!-- dept camra file  -->
   <xacro:include filename="dept_camera.xacro"/>

File: install/robot/share/robot/description/robot.urdf.xacro (robot description, xacro)
@@ -1,4 +1,11 @@
 <?xml version="1.0"?>
 <robot xmlns:xacro="http://www.ros.org/wiki/xacro" name="robot">
+  <!-- The robot .xacro file  -->
   <xacro:include filename="robot.xacro"/>
+  <!-- The gazebo control file  -->
+  <xacro:include filename="gazebo_controller.xacro"/>
+  <!-- The lidar sensor file  -->
+  <xacro:include filename="lidar_sensor.xacro"/>
+  <!-- dept camra file  -->
+  <xacro:include filename="dept_camera.xacro"/>
 </robot>

File: install/robot/share/robot/description/robot.xacro (robot description, xacro)
@@ -1,121 +1,127 @@
 <?xml version="1.0"?>
-<robot xmlns:xacro="http://www.ros.org/wiki/xacro" name="robot">
-<xacro:include filename="inertial.xacro"/>
- <!-- Setting the meshes colour  -->
-<!-- white -->
- <material name="white">
-    <color rgba="1 1 1 1" />
- </material>
- <!-- orange -->
- <material name="orange">
-    <color rgba="1 0.3 0.1 1" />
- </material>
- <!-- blue -->
- <material name="blue">
-    <color rgba="0.2 0.2 1 1" />
- </material>
- <!-- black -->
- <material name="black">
-    <color rgba="0 0 0 1" />
- </material>
-<!-- The link to the centre of the robot (called it "base_link") -->
-<link name="base_link">
-</link>
-<!-- link to the chassis  -->
-<joint name="chassis_joint" type="fixed">
-    <parent link="base_link"/>
-    <child link="chassis"/>
-<!-- We want the origin of the chassis sitting at the back/centre of the chassis -->
-    <origin xyz="-0.1 0 0"/>
-</joint>
-<link name="chassis">
-    <visual>
-        <origin xyz="0.15 0 0.075"/>
-        <geometry>
-            <box size="0.3 0.3 0.15"/>
-        </geometry>
-        <material name="orange"/>
-    </visual>
-    <collusion>
-        <origin xyz="0.15 0 0.075"/>
-        <geometry>
-            <box size="0.3 0.3 0.15"/>
-        </geometry>
-    </collusion>
-    <xacro:inertial_box mass="0.5" x="0.3" y="0.3" z="0.15">
-     <origin xyz="0.15 0 0.075" rpy="0 0 0"/>
-    </xacro:inertial_box>
-</link>
-<!-- The left wheel link  -->
-<joint name="left_wheel_joint" type="continuous">
-  <parent link="base_link"/>
-  <child link="left_wheel"/>
-  <origin xyz="0 0.175 0" rpy="-${pi/2} 0 0"/>
-  <axis xyz="0 0 1"/>
-</joint>
-<link name="left_wheel">
- <visual>
-    <geometry>
-       <cylinder radius="0.05" length="0.04"/>
-    </geometry>
-    <material name="black"/>
- </visual>
- <collusion>
-    <geometry>
-       <cylinder radius="0.05" length="0.04"/>
-    </geometry>
-    <material name="black"/>
- </collusion>
- <xacro:inertial_cylinder mass="0.1" length="0.04" radius="0.05">
-  <origin xyz="0 0 0" rpy="0 0 0"/>
- </xacro:inertial_cylinder>
-</link>
-<!-- The right wheel link  -->
-<joint name="right_wheel_joint" type="continuous">
-  <parent link="base_link"/>
-  <child link="right_wheel"/>
-  <origin xyz="0 -0.175 0" rpy="${pi/2} 0 0"/>
-  <axis xyz="0 0 -1"/>
-</joint>
-<link name="right_wheel">
- <visual>
-    <geometry>
-       <cylinder radius="0.05" length="0.04"/>
-    </geometry>
-    <material name="black"/>
- </visual>
- <collusion>
-    <geometry>
-       <cylinder radius="0.05" length="0.04"/>
-    </geometry>
- </collusion>
- <xacro:inertial_cylinder mass="0.1" length="0.04" radius="0.05">
-  <origin xyz="0 0 0" rpy="0 0 0"/>
- </xacro:inertial_cylinder>
-</link>
-<!-- dolly wheel link  -->
-<joint name="dolly_wheel_joint" type="fixed">
- <parent link="chassis"/>
- <child link="dolly_wheel"/>
- <origin xyz="0.24 0 0"/>
-</joint>
-<link name="dolly_wheel">
-<visual>
- <geometry>
-   <sphere radius="0.05"/>
- </geometry>
- <!-- give it a colour -->
- <material name="black"/>
-</visual>
-<collusion>
- <geometry>
-   <sphere radius="0.05"/>
- </geometry>
- <!-- give it a colour -->
- <material name="black"/>
-</collusion>
-<xacro:inertial_sphere mass="0.1"  radius="0.05">
-  <origin xyz="0 0 0" rpy="0 0 0"/>
- </xacro:inertial_sphere>
-</link>
+<robot xmlns:xacro="http://www.ros.org/wiki/xacro" >
+    <xacro:include filename="inertial.xacro"/>
+    <material name="white">
+        <color rgba="1 1 1 1" />
+    </material>
+    <material name="orange">
+        <color rgba="1 0.3 0.1 1"/>
+    </material>
+    <material name="blue">
+        <color rgba="0.2 0.2 1 1"/>
+    </material>
+    <material name="black">
+        <color rgba="0 0 0 1"/>
+    </material>
+    <!-- BASE LINK -->
+    <link name="base_link">
+    </link>
+    <!-- CHASSIS LINK -->
+    <joint name="chassis_joint" type="fixed">
+        <parent link="base_link"/>
+        <child link="chassis"/>
+        <origin xyz="-0.1 0 0"/>
+    </joint>
+    <link name="chassis">
+        <visual>
+            <origin xyz="0.15 0 0.075"/>
+            <geometry>
+                <box size="0.3 0.3 0.15"/>
+            </geometry>
+            <material name="blue"/>
+        </visual>
+        <collision>
+            <origin xyz="0.15 0 0.075"/>
+            <geometry>
+                <box size="0.3 0.3 0.15"/>
+            </geometry>
+        </collision>
+        <xacro:inertial_box mass="0.5" x="0.3" y="0.3" z="0.15">
+            <origin xyz="0.15 0 0.075" rpy="0 0 0"/>
+        </xacro:inertial_box>
+    </link>
+   <!-- Adding colour/fixing the colours to our urdf robot -->
+    <!-- chassis link colour (Adding chassis link colour) -->
+    <gazebo reference="chassis">
+      <material>Gazebo/Blue</material>
+    </gazebo>
+    <!-- LEFT WHEEL OF ROBOT -->
+    <joint name="left_wheel_joint" type="continuous">
+        <parent link="base_link"/>
+        <child link="left_wheel"/>
+        <origin xyz="0 0.175 0" rpy="-${pi/2} 0 0" />
+        <axis xyz="0 0 1"/>
+    </joint>
+    <link name="left_wheel">
+        <visual>
+            <geometry>
+                <cylinder radius="0.05" length="0.04"/>
+            </geometry>
+            <material name="black"/>
+        </visual>
+        <collision>
+            <geometry>
+                <cylinder radius="0.05" length="0.04"/>
+            </geometry>
+        </collision>
+        <xacro:inertial_cylinder mass="0.1" length="0.04" radius="0.05">
+            <origin xyz="0 0 0" rpy="0 0 0"/>
+        </xacro:inertial_cylinder>
+    </link>
+    <gazebo reference="left_wheel">
+      <material>Gazebo/Black</material>
+    </gazebo>
+    <!-- RIGHT WHEEL OF ROBOT -->
+    <joint name="right_wheel_joint" type="continuous">
+        <parent link="base_link"/>
+        <child link="right_wheel"/>
+        <origin xyz="0 -0.175 0" rpy="${pi/2} 0 0" />
+        <axis xyz="0 0 -1"/>
+    </joint>
+    <link name="right_wheel">
+        <visual>
+            <geometry>
+                <cylinder radius="0.05" length="0.04"/>
+            </geometry>
+            <material name="black"/>
+        </visual>
+        <collision>
+            <geometry>
+                <cylinder radius="0.05" length="0.04"/>
+            </geometry>
+        </collision>
+        <xacro:inertial_cylinder mass="0.1" length="0.04" radius="0.05">
+            <origin xyz="0 0 0" rpy="0 0 0"/>
+        </xacro:inertial_cylinder>
+    </link>
+     <gazebo reference="right_wheel">
+      <material>Gazebo/Black</material>
+    </gazebo>
+    <!-- DOLLY WHEEEL JOINT -->
+    <joint name="dolly_wheel_joint" type="fixed">
+        <parent link="chassis"/>
+        <child link="dolly_wheel"/>
+        <origin xyz="0.24 0 0"/>
+    </joint>
+    <link name="dolly_wheel">
+        <visual>
+            <geometry>
+                <sphere radius="0.05"/>
+            </geometry>`
+            <material name="black"/>
+        </visual>
+        <collision>
+            <geometry>
+                <sphere radius="0.05"/>
+            </geometry>
+        </collision>
+        <xacro:inertial_sphere mass="0.1" radius="0.05">
+            <origin xyz="0 0 0" rpy="0 0 0"/>
+        </xacro:inertial_sphere>
+    </link>
+     <gazebo reference="dolly_wheel">
+      <material>Gazebo/Black</material>
+      <mu1 value="0.100"/>
+      <mu2 value="0.100"/>
+    </gazebo>
 </robot>
